File: 5vSwitcher.sch (EAGLE design)
At the start: 5 parts, among them IC1 LM2596S

Commit message: Added notice
Parts:
- D1: value (none) -> 1N5822
- L1: value (none) -> 100uH
Other:
- note added: "Reference Designs ARE PROVIDED "AS IS" AND "WITH ALL FAULTS.Black Electronics DISCLAIMS ALL OTHER WARRANTIES, EXPRESS OR IMPLIED,REGARDING PRODUCTS, INCLUDING BUT NOT LIMITED TO, ANY IMPLIED WARRANTIESOF MERCHANTABILITY OR FITNESS FOR A PARTICULAR PURPOSE Black Electronics may make changes to specifications and product description at any time, without notice. The customer must not rely on the abs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"
Changed lines of the file:
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@@
 <part name="IC1" library="national-semiconductor" deviceset="LM2596" device="S"/>
 <part name="JP1" library="SparkFun" deviceset="M03" device="PTH"/>
-<part name="D1" library="diode" deviceset="SCHOTTKY-DIODE" device="SMC"/>
-<part name="L1" library="SparkFun" deviceset="INDUCTOR" device="H*" technology="1206"/>
+<part name="D1" library="diode" deviceset="SCHOTTKY-DIODE" device="SMC" value="1N5822"/>
+<part name="L1" library="SparkFun" deviceset="INDUCTOR" device="H*" technology="1206" value="100uH"/>
 </parts>
 <sheets>
 <sheet>
 <plain>
+<text x="2.54" y="-20.32" size="1.778" layer="91">Reference Designs ARE PROVIDED "AS IS" AND "WITH ALL FAULTS.Black Electronics DISCLAIMS ALL OTHER WARRANTIES, EXPRESS
+OR IMPLIED,REGARDING PRODUCTS, INCLUDING BUT NOT LIMITED TO, ANY IMPLIED WARRANTIESOF MERCHANTABILITY OR FITNESS
+FOR A PARTICULAR PURPOSE Black Electronics may make changes to specifications and product description at any time, without notice.
+The customer must not rely on the absence or characterics of any feature or instruction marked "reserved" or "undefined".
+Black Electronics reserves these for future definition and shall have no responsibility whatsoever for the conflicts or
+incompatibilities arsing from future changes to them. The product information on the Web Site or Materials is subject to change without notice.
+Do not finalize  design with this information.</text>
 </plain>
 <instances>
@@
 </schematic>
 </drawing>
+<compatibility>
+<note version="6.3" minversion="6.2.2" severity="warning">
+Since Version 6.2.2 text objects can contain more than one line,
+which will not be processed correctly with this version.
+</note>
+</compatibility>
 </eagle>

Commit message: Clean up
Parts:
- added C1, C2: 100uF, SparkFun:CAP0805
Connections:
- net GND: now also C1.2, C2.2
- net VOUT: now also C1.1, C2.1
Other:
- note added: "Reference Designs ARE PROVIDED "AS IS" AND "WITH ALL FAULTS. Black Electronics DISCLAIMS ALL OTHER WARRANTIES, EXPRESS OR IMPLIED, REGARDING PRODUCTS, INCLUDING BUT NOT LIMITED TO, ANY IMPLIED WARRANTIESOF MERCHANTABILITY OR FITNESS FOR A PARTICULAR PURPOSE Black Electronics may make changes to specifications and product description at any time, without notice. The customer must not rely on the a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"
- note removed: "Reference Designs ARE PROVIDED "AS IS" AND "WITH ALL FAULTS.Black Electronics DISCLAIMS ALL OTHER WARRANTIES, EXPRESS OR IMPLIED,REGARDING PRODUCTS, INCLUDING BUT NOT LIMITED TO, ANY IMPLIED WARRANTIESOF MERCHANTABILITY OR FITNESS FOR A PARTICULAR PURPOSE Black Electronics may make changes to specifications and product description at any time, without notice. The customer must not rely on the abs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"
- moved on the sheet: D1
Changed lines of the file:
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@@
 <part name="D1" library="diode" deviceset="SCHOTTKY-DIODE" device="SMC" value="1N5822"/>
 <part name="L1" library="SparkFun" deviceset="INDUCTOR" device="H*" technology="1206" value="100uH"/>
+<part name="C1" library="SparkFun" deviceset="CAP" device="0805" value="100uF"/>
+<part name="C2" library="SparkFun" deviceset="CAP" device="0805" value="100uF"/>
 </parts>
 <sheets>
 <sheet>
 <plain>
-<text x="2.54" y="-20.32" size="1.778" layer="91">Reference Designs ARE PROVIDED "AS IS" AND "WITH ALL FAULTS.Black Electronics DISCLAIMS ALL OTHER WARRANTIES, EXPRESS
-OR IMPLIED,REGARDING PRODUCTS, INCLUDING BUT NOT LIMITED TO, ANY IMPLIED WARRANTIESOF MERCHANTABILITY OR FITNESS
+<text x="2.54" y="-20.32" size="1.778" layer="91">Reference Designs ARE PROVIDED "AS IS" AND "WITH ALL FAULTS. Black Electronics DISCLAIMS ALL OTHER WARRANTIES, EXPRESS
+OR IMPLIED, REGARDING PRODUCTS, INCLUDING BUT NOT LIMITED TO, ANY IMPLIED WARRANTIESOF MERCHANTABILITY OR FITNESS
 FOR A PARTICULAR PURPOSE Black Electronics may make changes to specifications and product description at any time, without notice.
 The customer must not rely on the absence or characterics of any feature or instruction marked "reserved" or "undefined".
 Black Electronics reserves these for future definition and shall have no responsibility whatsoever for the conflicts or
 incompatibilities arsing from future changes to them. The product information on the Web Site or Materials is subject to change without notice.
-Do not finalize  design with this information.</text>
+Do not finalize design with this information.</text>
 </plain>
 <instances>
@@
 <instance part="IC1" gate="G$1" x="99.06" y="116.84"/>
 <instance part="JP1" gate="G$1" x="193.04" y="119.38" rot="R180"/>
-<instance part="D1" gate="G$1" x="114.3" y="104.14" rot="R90"/>
+<instance part="D1" gate="G$1" x="114.3" y="106.68" rot="R90"/>
 <instance part="L1" gate="G$1" x="127" y="119.38" rot="R90"/>
+<instance part="C1" gate="G$1" x="147.32" y="109.22"/>
+<instance part="C2" gate="G$1" x="157.48" y="109.22"/>
 </instances>
 <busses>
@@
 <net name="GND" class="0">
 <segment>
+<pinref part="C1" gate="G$1" pin="2"/>
+<wire x1="147.32" y1="101.6" x2="147.32" y2="106.68" width="0.1524" layer="91"/>
+<pinref part="IC1" gate="G$1" pin="!ON!/OFF"/>
+<wire x1="83.82" y1="116.84" x2="86.36" y2="116.84" width="0.1524" layer="91"/>
 <pinref part="IC1" gate="G$1" pin="GND"/>
 <wire x1="86.36" y1="111.76" x2="83.82" y2="111.76" width="0.1524" layer="91"/>
@@
 <wire x1="83.82" y1="111.76" x2="83.82" y2="116.84" width="0.1524" layer="91"/>
 <junction x="83.82" y="111.76"/>
-<pinref part="IC1" gate="G$1" pin="!ON!/OFF"/>
-<wire x1="83.82" y1="116.84" x2="86.36" y2="116.84" width="0.1524" layer="91"/>
+<wire x1="83.82" y1="101.6" x2="83.82" y2="111.76" width="0.1524" layer="91"/>
 <label x="76.2" y="111.76" size="1.778" layer="95"/>
-<wire x1="114.3" y1="101.6" x2="83.82" y2="101.6" width="0.1524" layer="91"/>
-<wire x1="83.82" y1="101.6" x2="83.82" y2="111.76" width="0.1524" layer="91"/>
+<wire x1="83.82" y1="101.6" x2="114.3" y2="101.6" width="0.1524" layer="91"/>
 <pinref part="D1" gate="G$1" pin="A"/>
+<wire x1="114.3" y1="101.6" x2="147.32" y2="101.6" width="0.1524" layer="91"/>
+<wire x1="114.3" y1="104.14" x2="114.3" y2="101.6" width="0.1524" layer="91"/>
+<junction x="114.3" y="101.6"/>
+<pinref part="C2" gate="G$1" pin="2"/>
+<wire x1="147.32" y1="101.6" x2="157.48" y2="101.6" width="0.1524" layer="91"/>
+<wire x1="157.48" y1="101.6" x2="157.48" y2="106.68" width="0.1524" layer="91"/>
+<junction x="147.32" y="101.6"/>
 </segment>
 <segment>
@@
 <pinref part="IC1" gate="G$1" pin="OUT"/>
 <wire x1="114.3" y1="119.38" x2="111.76" y2="119.38" width="0.1524" layer="91"/>
-<wire x1="114.3" y1="106.68" x2="114.3" y2="119.38" width="0.1524" layer="91"/>
+<wire x1="114.3" y1="109.22" x2="114.3" y2="119.38" width="0.1524" layer="91"/>
 <pinref part="L1" gate="G$1" pin="1"/>
 <wire x1="114.3" y1="119.38" x2="119.38" y2="119.38" width="0.1524" layer="91"/>
@@
 <wire x1="111.76" y1="114.3" x2="144.78" y2="114.3" width="0.1524" layer="91"/>
 <wire x1="144.78" y1="114.3" x2="144.78" y2="119.38" width="0.1524" layer="91"/>
-<wire x1="144.78" y1="119.38" x2="154.94" y2="119.38" width="0.1524" layer="91"/>
-<label x="149.86" y="119.38" size="1.778" layer="95"/>
+<wire x1="144.78" y1="119.38" x2="147.32" y2="119.38" width="0.1524" layer="91"/>
+<label x="157.48" y="119.38" size="1.778" layer="95"/>
 <pinref part="L1" gate="G$1" pin="2"/>
+<wire x1="147.32" y1="119.38" x2="157.48" y2="119.38" width="0.1524" layer="91"/>
 <wire x1="134.62" y1="119.38" x2="144.78" y2="119.38" width="0.1524" layer="91"/>
 <junction x="144.78" y="119.38"/>
+<pinref part="C1" gate="G$1" pin="1"/>
+<wire x1="147.32" y1="114.3" x2="147.32" y2="119.38" width="0.1524" layer="91"/>
+<junction x="147.32" y="119.38"/>
+<pinref part="C2" gate="G$1" pin="1"/>
+<wire x1="157.48" y1="114.3" x2="157.48" y2="119.38" width="0.1524" layer="91"/>
+<wire x1="157.48" y1="119.38" x2="162.56" y2="119.38" width="0.1524" layer="91"/>
+<junction x="157.48" y="119.38"/>
 </segment>
 <segment>
